File: pcb/sensor_module_carrier.kicad_pcb (KiCad board)
At the start: 2 copper layers, 49 x 23 mm, 5 parts, among them J1 Conn_01x04_Pin, J2 HCTL HC-SFP-20P

Commit message: v2
Parts:
- moved H1 2.60 mm to (103.9, 70.2)
- moved H2 2.60 mm to (86.8, 76.2)
- moved H3 2.60 mm to (103.9, 82.2)
Other:
- board size 49 x 23 mm -> 48 x 23 mm
- board text added: "test v2"
- board text removed: "test v1"
Changed lines of the file:
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@@
 	(footprint "Mounting_Wuerth:Mounting_Wuerth_WA-SMSI-M2.5_H2.5mm_9774025151R"
 		(layer "F.Cu")
-		(at 106.5 82.2)
+		(at 103.904127 82.2)
 		(descr "Mounting Hardware, inside through hole M2.5, height 2.5, Wuerth electronics 9774025151R (https://www.we-online.com/components/products/datasheet/9774025151R.pdf), generated with kicad-footprint-generator")
 		(tags "Mounting M2.5 9774025151R")
@@
 	(footprint "Mounting_Wuerth:Mounting_Wuerth_WA-SMSI-M2.5_H2.5mm_9774025151R"
 		(layer "F.Cu")
-		(at 106.5 70.2)
+		(at 103.904127 70.2)
 		(descr "Mounting Hardware, inside through hole M2.5, height 2.5, Wuerth electronics 9774025151R (https://www.we-online.com/components/products/datasheet/9774025151R.pdf), generated with kicad-footprint-generator")
 		(tags "Mounting M2.5 9774025151R")
@@
 	(footprint "Mounting_Wuerth:Mounting_Wuerth_WA-SMSI-M2.5_H2.5mm_9774025151R"
 		(layer "F.Cu")
-		(at 89.425 76.2)
+		(at 86.829127 76.2)
 		(descr "Mounting Hardware, inside through hole M2.5, height 2.5, Wuerth electronics 9774025151R (https://www.we-online.com/components/products/datasheet/9774025151R.pdf), generated with kicad-footprint-generator")
 		(tags "Mounting M2.5 9774025151R")
@@
 	)
 	(gr_line
-		(start 108.5 65.2)
-		(end 108.5 84.2)
-		(stroke
-			(width 0.15)
-			(type default)
-		)
-		(layer "F.SilkS")
-	)
-	(gr_line
 		(start 88.5 65.2)
 		(end 88.5 87.2)
@@
 	)
 	(gr_line
-		(start 107.5 74.2)
-		(end 107.5 78.2)
+		(start 105 74.2)
+		(end 105 78.2)
 		(stroke
 			(width 0.15)
@@
 	)
 	(gr_line
-		(start 108.5 74.2)
-		(end 108.5 78.2)
+		(start 106 74.2)
+		(end 106 78.2)
+		(stroke
+			(width 0.15)
+			(type default)
+		)
+		(layer "F.SilkS")
+	)
+	(gr_line
+		(start 107 74.2)
+		(end 107 78.2)
 		(stroke
 			(width 0.15)
@@
 	)
 	(gr_line
-		(start 106.5 74.2)
-		(end 106.5 78.2)
-		(stroke
-			(width 0.15)
-			(type default)
-		)
-		(layer "F.SilkS")
-	)
-	(gr_line
-		(start 109.5 65.2)
-		(end 109.5 87.2)
+		(start 104 74.2)
+		(end 104 78.2)
 		(stroke
 			(width 0.15)
@@
 	)
 	(gr_line
-		(start 86.5 86.2)
-		(end 109 86.2)
+		(start 108 74.2)
+		(end 108 78.2)
+		(stroke
+			(width 0.15)
+			(type default)
+		)
+		(layer "F.SilkS")
+	)
+	(gr_line
+		(start 84 86.2)
+		(end 106.5 86.2)
 		(stroke
 			(width 0.1)
@@
 	)
 	(gr_line
-		(start 109 66.2)
-		(end 86.5 66.2)
+		(start 106.5 66.2)
+		(end 84 66.2)
 		(stroke
 			(width 0.1)
@@
 	)
 	(gr_line
-		(start 86.5 81.8)
-		(end 86.5 86.2)
+		(start 84 81.8)
+		(end 84 86.2)
 		(stroke
 			(width 0.1)
@@
 	)
 	(gr_arc
-		(start 85.5 80.8)
-		(mid 86.207107 81.092893)
-		(end 86.5 81.8)
+		(start 83 80.8)
+		(mid 83.707107 81.092893)
+		(end 84 81.8)
 		(stroke
 			(width 0.1)
@@
 	)
 	(gr_arc
-		(start 86.5 70.6)
-		(mid 86.207107 71.307107)
-		(end 85.5 71.6)
+		(start 84 70.6)
+		(mid 83.707107 71.307107)
+		(end 83 71.6)
 		(stroke
 			(width 0.1)
@@
 	)
 	(gr_line
-		(start 86.5 70.6)
-		(end 86.5 66.2)
+		(start 84 70.6)
+		(end 84 66.2)
 		(stroke
 			(width 0.1)
@@
 	)
 	(gr_line
-		(start 85 71.6)
-		(end 85.5 71.6)
+		(start 82.5 71.6)
+		(end 83 71.6)
 		(stroke
 			(width 0.1)
@@
 	)
 	(gr_line
-		(start 85 80.8)
-		(end 85.5 80.8)
+		(start 82.5 80.8)
+		(end 83 80.8)
 		(stroke
 			(width 0.1)
@@
 	)
 	(gr_line
-		(start 109 86.2)
-		(end 109 66.2)
+		(start 106.5 86.2)
+		(end 106.5 66.2)
 		(stroke
 			(width 0.1)
@@
 	(gr_rect
 		(start 61 64.7)
-		(end 110 87.7)
+		(end 109 87.7)
 		(stroke
 			(width 0.1)
@@
 	)
 	(gr_text "JLCJLCJLCJLC"
-		(at 93 74.7 0)
+		(at 93 76.75 0)
 		(layer "F.SilkS")
 		(effects
@@
 		)
 	)
-	(gr_text "test v1"
+	(gr_text "test v2"
 		(at 77.5 67.2 0)
 		(layer "F.SilkS")
