File: pcb/sensor_module_carrier.kicad_sch (KiCad schematic)
At the start: 5 parts, among them J1 Conn_01x04_Pin, J2 HCTL HC-SFP-20P

Commit message: v2
Other:
- moved on the sheet: H3
Changed lines of the file:
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@@
 	(symbol
 		(lib_id "Mechanical:MountingHole")
-		(at 80.01 96.52 0)
+		(at 80.01 95.25 0)
 		(unit 1)
 		(exclude_from_sim no)
@@
 		(fields_autoplaced yes)
 		(property "Reference" "H3"
-			(at 82.55 95.885 0)
+			(at 82.55 94.615 0)
 			(effects
 				(font
@@
 		)
 		(property "Value" "SMSI-M2_H4mm_9774040243"
-			(at 82.55 98.425 0)
+			(at 82.55 97.155 0)
 			(effects
 				(font
@@
 		)
 		(property "Footprint" "Mounting_Wuerth:Mounting_Wuerth_WA-SMSI-M2.5_H2.5mm_9774025151R"
-			(at 80.01 96.52 0)
+			(at 80.01 95.25 0)
 			(effects
 				(font
@@
 		)
 		(property "Datasheet" "~"
-			(at 80.01 96.52 0)
+			(at 80.01 95.25 0)
 			(effects
 				(font
@@
 		)
 		(property "Description" ""
-			(at 80.01 96.52 0)
+			(at 80.01 95.25 0)
 			(effects
 				(font
@@
 		)
 		(property "LCSC" ""
-			(at 80.01 96.52 0)
+			(at 80.01 95.25 0)
 			(effects
 				(font
@@
 		)
 		(property "Notes" ""
-			(at 80.01 96.52 0)
+			(at 80.01 95.25 0)
 			(effects
 				(font
