File: modules/hybrid/hybrid.kicad_sch (KiCad schematic)
At the start: 5 parts, among them J1 SensorModule, U1 SDP810

Commit message: Hybrid sensor module, SDP810 screw mounts (interface-v3), main board J6 adoption
Hybrid module (modules/hybrid): one L42 board that takes either an SDP810 (U1)
or an XGZP6899D (U2) on a shared site at 22 mm; fit one, never both. The SDP810
is screwed down through its body bores (M2x14, Ø2.2 NPTH) into carrier nuts at
10 and 34 mm, with B-side keepouts there. J2 is a bottom-side 1x5 pogo test pad
row, GND-SCL-3V3-SDA-GND, so a reversed jig only swaps SDA/SCL. Corners R1.

Interface v3: carrier nuts at 2.925, 10, 34 and 40 mm; the 30 mm nut is gone
(it overlaps 34 mm), which retires L32 and the xgzp6899 module. New shared
footprint sensor_module:TestPads_1x05_P2.54mm. Skeleton keepouts moved to 10/34.

Main board: J6 wired up, H7 moved to 34 mm and H9 added at 10 mm, R13 5k1
pull-up on GPIO4 (shared ~SPI_CS / UART_P2C).

Removed the breakout carrier; module CI now only scans modules/ and skips
the skeleton template.
Parts:
- added J2: Pogo test pads, sensor_module:TestPads_1x05_P2.54mm, symbol Connector_Generic:Conn_01x05
- added U2: XGZP6899D, Sensor_Pressure:CFSensor_XGZP6899x, symbol Sensor_Pressure:XGZP6899D
- C1: now not fitted
Connections:
- net +3V3: now also J2.3 (Pin_3), U2.6 (VDD)
- net GND: now also J2.1 (Pin_1), J2.5 (Pin_5), U2.2 (GND)
- net SCL: now also J2.2 (Pin_2), U2.3 (SCL)
- net SDA: now also J2.4 (Pin_4), U2.4 (SDA)
Other:
- note added: "Fit U1 (SDP810) OR U2 (XGZP6899D), never both: the footprints overlap on the PCB. I2C: SDP810 0x25, XGZP6899D 0x6D"
- note added: "Pogo test pads (module bottom)"
- title: serialsentinel -> hybrid sensor module
